File: Hardware/projects/Current-KiCAD-Design/WIBL.kicad_pcb (KiCad board)
At the start: 2 copper layers, 110 x 56 mm, 112 parts, among them IC1 SN65C1168N, J1 N2K 5-PIN, T1 S8050, T2 S8050, T3 S8050, T4 S8050, U1 ESP32-WROOM-32E-N4, U2 TJA1051T/3, U3 LSM6DS3TR-C, U4 AMS1117-3.3, U6 RFM-0505S, U7 LV2842XLVDDCR

Commit message: HW: Updates for 2.5.1 hardware release using KiCAD files.
Connections:
- OK1 pad 3: (no net) -> unconnected-(OK1-NC-Pad3)
- OK2 pad 3: (no net) -> unconnected-(OK2-NC-Pad3)
- OK3 pad 3: (no net) -> unconnected-(OK3-NC-Pad3)
- OK4 pad 3: (no net) -> unconnected-(OK4-NC-Pad3)
Changed lines of the file:
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@@
 	(net 79 "Net-(IC1-2D)")
 	(net 80 "unconnected-(U4-Tab-Pad4)")
+	(net 81 "unconnected-(OK3-NC-Pad3)")
+	(net 82 "unconnected-(OK4-NC-Pad3)")
+	(net 83 "unconnected-(OK1-NC-Pad3)")
+	(net 84 "unconnected-(OK2-NC-Pad3)")
 	(footprint "WIBL:R0805_334"
 		(layer "F.Cu")
@@
 		(sheetname "/")
 		(sheetfile "WIBL.kicad_sch")
+		(attr exclude_from_bom)
 		(fp_circle
 			(center 0 0)
@@
 			(pinfunction "1")
 			(pintype "passive")
-			(clearance 0.8)
 			(zone_connect 2)
 		)
@@
 			(pinfunction "1")
 			(pintype "passive")
-			(clearance 0.8)
 			(zone_connect 2)
 		)
@@
 		(sheetname "/")
 		(sheetfile "WIBL.kicad_sch")
+		(attr exclude_from_bom)
 		(fp_circle
 			(center 0 0)
@@
 		(descr "DIL 6 SMD\n\nSource: http://www.fairchildsemi.com/pf/4N/4N35-M.html")
 		(property "Reference" "OK2"
-			(at -4.8961 8.8391 0)
+			(at -3.36195 2 270)
 			(unlocked yes)
 			(layer "F.SilkS")
 			(effects
 				(font
-					(size 1 1)
+					(size 1.143 1.143)
 					(thickness 0.1524)
 				)
@@
 		)
 		(property "Value" "H11L1SM"
-			(at -3.81 0.635 270)
+			(at -4.2061 -1.4709 270)
 			(unlocked yes)
-			(layer "F.Fab")
-			(hide yes)
+			(layer "F.SilkS")
 			(effects
 				(font
 					(size 1.143 1.143)
-					(thickness 0.127)
+					(thickness 0.1524)
 				)
-				(justify right top)
+				(justify left bottom)
 			)
 		)
@@
 		)
 		(property "Mfr" "Isocom Components 2004 LTD"
-			(at 0 0 270)
+			(at 0 0 90)
 			(layer "F.SilkS")
 			(hide yes)
@@
 		)
 		(property "MPNum" "H11L1SM"
-			(at 0 0 270)
+			(at 0 0 90)
 			(layer "F.SilkS")
 			(hide yes)
@@
 			(size 1.78 1.52)
 			(layers "F.Cu" "F.Mask" "F.Paste")
+			(net 84 "unconnected-(OK2-NC-Pad3)")
+			(pinfunction "NC")
+			(pintype "no_connect")
 			(solder_mask_margin 0.1016)
 			(thermal_bridge_angle 0)
@@
 		(descr "DIL 6 SMD\n\nSource: http://www.fairchildsemi.com/pf/4N/4N35-M.html")
 		(property "Reference" "OK4"
-			(at -3.6 -5.8391 0)
+			(at -3.36195 2 90)
 			(unlocked yes)
 			(layer "F.SilkS")
 			(effects
 				(font
-					(size 1 1)
+					(size 1.143 1.143)
 					(thickness 0.1524)
 				)
-				(justify right top)
+				(justify left bottom)
 			)
 		)
 		(property "Value" "H11L1SM"
-			(at -3.81 0.635 90)
+			(at -3.81 -1.2391 90)
 			(unlocked yes)
-			(layer "F.Fab")
-			(hide yes)
+			(layer "F.SilkS")
 			(effects
 				(font
 					(size 1.143 1.143)
-					(thickness 0.127)
+					(thickness 0.1524)
 				)
-				(justify right top)
+				(justify left bottom)
 			)
 		)
@@
 			(size 1.78 1.52)
 			(layers "F.Cu" "F.Mask" "F.Paste")
+			(net 82 "unconnected-(OK4-NC-Pad3)")
+			(pinfunction "NC")
+			(pintype "no_connect")
 			(solder_mask_margin 0.1016)
 			(thermal_bridge_angle 0)
@@
 		(sheetname "/")
 		(sheetfile "WIBL.kicad_sch")
+		(attr exclude_from_bom)
 		(fp_circle
 			(center 0 0)
@@
 			(pinfunction "1")
 			(pintype "passive")
-			(clearance 0.8)
 			(zone_connect 2)
 		)
@@
 			(pinfunction "1")
 			(pintype "passive")
-			(clearance 0.8)
 			(zone_connect 2)
 		)
@@
 		(descr "DIL 6 SMD\n\nSource: http://www.fairchildsemi.com/pf/4N/4N35-M.html")
 		(property "Reference" "OK1"
-			(at -4.7 8.5391 0)
+			(at -3.36195 2 270)
 			(unlocked yes)
 			(layer "F.SilkS")
 			(effects
 				(font
-					(size 1 1)
+					(size 1.143 1.143)
 					(thickness 0.1524)
 				)
@@
 		)
 		(property "Value" "H11L1SM"
-			(at -3.81 0.635 270)
+			(at -4.13 -1.2709 270)
 			(unlocked yes)
-			(layer "F.Fab")
-			(hide yes)
+			(layer "F.SilkS")
 			(effects
 				(font
 					(size 1.143 1.143)
-					(thickness 0.127)
+					(thickness 0.1524)
 				)
-				(justify right top)
+				(justify left bottom)
 			)
 		)
@@
 			(size 1.78 1.52)
 			(layers "F.Cu" "F.Mask" "F.Paste")
+			(net 83 "unconnected-(OK1-NC-Pad3)")
+			(pinfunction "NC")
+			(pintype "no_connect")
 			(solder_mask_margin 0.1016)
 			(thermal_bridge_angle 0)
@@
 		(descr "DIL 6 SMD\n\nSource: http://www.fairchildsemi.com/pf/4N/4N35-M.html")
 		(property "Reference" "OK3"
-			(at -9.9 -6.3247 0)
+			(at -3.36195 2 90)
 			(unlocked yes)
 			(layer "F.SilkS")
 			(effects
 				(font
-					(size 1 1)
+					(size 1.143 1.143)
 					(thickness 0.1524)
 				)
-				(justify right top)
+				(justify left bottom)
 			)
 		)
 		(property "Value" "H11L1SM"
-			(at -3.81 0.635 90)
+			(at -4.37 -1.4691 90)
 			(unlocked yes)
-			(layer "F.Fab")
-			(hide yes)
+			(layer "F.SilkS")
 			(effects
 				(font
 					(size 1.143 1.143)
-					(thickness 0.127)
+					(thickness 0.1524)
 				)
-				(justify right top)
+				(justify left bottom)
 			)
 		)
@@
 			(size 1.78 1.52)
 			(layers "F.Cu" "F.Mask" "F.Paste")
+			(net 81 "unconnected-(OK3-NC-Pad3)")
+			(pinfunction "NC")
+			(pintype "no_connect")
 			(solder_mask_margin 0.1016)
 			(thermal_bridge_angle 0)
@@
 		(sheetname "/")
 		(sheetfile "WIBL.kicad_sch")
+		(attr exclude_from_bom)
 		(fp_circle
 			(center 0 0)
