File: Hardware/projects/Current-KiCAD-Design/WIBL.kicad_sch (KiCad schematic)
At the start: 7 parts

Commit message: HW: Updates for 2.5.1 hardware release using KiCAD files.
Parts:
- MH1, MH2, MH3, MH4: symbol EE_NON_BOM_250715:MTH_P_3.2mm_M3 -> WIBL-eagle-import:MTH_P_3.2mm_M3; now left out of the parts list
Changed lines of the file:
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@@
 	)
 	(symbol
-		(lib_id "EE_NON_BOM_250715:MTH_P_3.2mm_M3")
+		(lib_id "WIBL-eagle-import:MTH_P_3.2mm_M3")
 		(at 11.43 78.74 0)
 		(unit 1)
 		(exclude_from_sim no)
-		(in_bom yes)
+		(in_bom no)
 		(on_board yes)
 		(dnp no)
@@
 	)
 	(symbol
-		(lib_id "EE_NON_BOM_250715:MTH_P_3.2mm_M3")
+		(lib_id "WIBL-eagle-import:MTH_P_3.2mm_M3")
 		(at 49.53 78.74 0)
 		(unit 1)
 		(exclude_from_sim no)
-		(in_bom yes)
+		(in_bom no)
 		(on_board yes)
 		(dnp no)
@@
 	)
 	(symbol
-		(lib_id "EE_NON_BOM_250715:MTH_P_3.2mm_M3")
+		(lib_id "WIBL-eagle-import:MTH_P_3.2mm_M3")
 		(at 36.83 78.74 0)
 		(unit 1)
 		(exclude_from_sim no)
-		(in_bom yes)
+		(in_bom no)
 		(on_board yes)
 		(dnp no)
@@
 	)
 	(symbol
-		(lib_id "EE_NON_BOM_250715:MTH_P_3.2mm_M3")
+		(lib_id "WIBL-eagle-import:MTH_P_3.2mm_M3")
 		(at 24.13 78.74 0)
 		(unit 1)
 		(exclude_from_sim no)
-		(in_bom yes)
-		(on_board yes)
-		(dnp no)
+		(in_bom no)
+		(on_board yes)
+		(dnp no)
